File: Esquematicos/CAE32_PCB/Pedals/Pedals/Connectors.kicad_sch (KiCad schematic)
At the start: 8 parts, among them J15 USB_C_Receptacle_USB2.0, J16 UART_PGR, J17 ST-Link

Commit message: add: plantilla para diseño de pcb para shifter
Parts:
- removed J17: ST-Link, Connector_PinSocket_2.54mm:PinSocket_1x05_P2.54mm_Vertical, symbol Connector:Conn_01x05_Female
Other:
- note added: "Programming an Debugging port"
- note removed: "Programming an Debugging ports"
Changed lines of the file:
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@@
     (stroke (width 0) (type default) (color 0 0 0 0))
   )
-  (polyline (pts (xy 280.035 15.24) (xy 280.035 54.864))
+  (polyline (pts (xy 261.62 15.24) (xy 261.62 54.61))
     (stroke (width 0) (type default) (color 0 0 0 0))
   )
@@
     (stroke (width 0) (type default) (color 0 0 0 0))
   )
-  (polyline (pts (xy 224.79 54.864) (xy 280.035 54.864))
+  (polyline (pts (xy 224.79 54.864) (xy 261.62 54.61))
     (stroke (width 0) (type default) (color 0 0 0 0))
   )
@@
     (stroke (width 0) (type default) (color 0 0 0 0))
   )
-  (polyline (pts (xy 224.79 15.24) (xy 280.035 15.24))
+  (polyline (pts (xy 224.79 15.24) (xy 261.62 15.24))
     (stroke (width 0) (type default) (color 0 0 0 0))
   )
@@
     (stroke (width 0) (type default) (color 0 0 0 0))
   )
-  (wire (pts (xy 270.51 29.845) (xy 270.51 32.385))
-    (stroke (width 0) (type default) (color 0 0 0 0))
-  )
   (wire (pts (xy 73.914 50.8) (xy 87.122 50.8))
     (stroke (width 0) (type default) (color 0 0 0 0))
@@
     (stroke (width 0) (type default) (color 0 0 0 0))
   )
-  (wire (pts (xy 270.51 42.545) (xy 270.51 45.085))
-    (stroke (width 0) (type default) (color 0 0 0 0))
-  )
-  (text "Programming an\nDebugging ports" (at 243.205 20.955 0)
+  (text "Programming an\nDebugging port" (at 243.205 20.955 0)
     (effects (font (size 1.27 1.27)) (justify left bottom))
   )
@@
     (effects (font (size 1.27 1.27)) (justify left))
   )
-  (hierarchical_label "NRST" (shape input) (at 270.51 34.925 0)
-    (effects (font (size 1.27 1.27)) (justify left))
-  )
-  (hierarchical_label "SWDIO" (shape input) (at 270.51 37.465 0)
-    (effects (font (size 1.27 1.27)) (justify left))
-  )
   (hierarchical_label "PGR_UART_RX" (shape input) (at 242.57 38.735 0)
     (effects (font (size 1.27 1.27)) (justify left))
@@
     (effects (font (size 1.27 1.27)) (justify left))
   )
-  (hierarchical_label "SWCLK" (shape input) (at 270.51 40.005 0)
-    (effects (font (size 1.27 1.27)) (justify left))
-  )
   (hierarchical_label "D+" (shape input) (at 87.376 55.88 0)
     (effects (font (size 1.27 1.27)) (justify left))
@@
   (hierarchical_label "D+" (shape input) (at 87.376 53.34 0)
     (effects (font (size 1.27 1.27)) (justify left))
-  )
-  (symbol (lib_id "power:GNDREF") (at 270.51 45.085 0) (unit 1)
-    (in_bom yes) (on_board yes) (fields_autoplaced)
-    (property "Reference" "#PWR048" (id 0) (at 270.51 51.435 0)
-      (effects (font (size 1.27 1.27)) hide)
-    )
-    (property "Value" "GNDREF" (id 1) (at 270.51 50.165 0))
-    (property "Footprint" "" (id 2) (at 270.51 45.085 0)
-      (effects (font (size 1.27 1.27)) hide)
-    )
-    (property "Datasheet" "" (id 3) (at 270.51 45.085 0)
-      (effects (font (size 1.27 1.27)) hide)
-    )
-    (pin "1")
   )
   (symbol (lib_name "GNDREF_1") (lib_id "power:GNDREF") (at 76.454 70.866 0) (unit 1)
@@
     (pin "S1")
   )
-  (symbol (lib_id "power:+3.3V") (at 270.51 29.845 0) (unit 1)
-    (in_bom yes) (on_board yes) (fields_autoplaced)
-    (property "Reference" "#PWR047" (id 0) (at 270.51 33.655 0)
-      (effects (font (size 1.27 1.27)) hide)
-    )
-    (property "Value" "+3.3V" (id 1) (at 270.51 24.765 0))
-    (property "Footprint" "" (id 2) (at 270.51 29.845 0)
-      (effects (font (size 1.27 1.27)) hide)
-    )
-    (property "Datasheet" "" (id 3) (at 270.51 29.845 0)
-      (effects (font (size 1.27 1.27)) hide)
-    )
-    (pin "1")
-  )
   (symbol (lib_name "GNDREF_1") (lib_id "power:GNDREF") (at 74.93 43.18 0) (unit 1)
     (in_bom yes) (on_board yes)
@@
     (pin "2")
   )
-  (symbol (lib_id "Connector:Conn_01x05_Female") (at 265.43 37.465 180) (unit 1)
-    (in_bom yes) (on_board yes)
-    (property "Reference" "J17" (id 0) (at 264.16 38.7351 0)
-      (effects (font (size 1.27 1.27)) (justify left))
-    )
-    (property "Value" "ST-Link" (id 1) (at 264.16 36.1951 0)
-      (effects (font (size 1.27 1.27)) (justify left))
-    )
-    (property "Footprint" "Connector_PinSocket_2.54mm:PinSocket_1x05_P2.54mm_Vertical" (id 2) (at 265.43 37.465 0)
-      (effects (font (size 1.27 1.27)) hide)
-    )
-    (property "Datasheet" "~" (id 3) (at 265.43 37.465 0)
-      (effects (font (size 1.27 1.27)) hide)
-    )
-    (property "LCSC_PART" "C50950" (id 4) (at 265.43 37.465 0)
-      (effects (font (size 1.27 1.27)) hide)
-    )
-    (property "Item" "C50950" (id 5) (at 265.43 37.465 0)
-      (effects (font (size 1.27 1.27)) hide)
-    )
-    (property "Qty" "1" (id 6) (at 265.43 37.465 0)
-      (effects (font (size 1.27 1.27)) hide)
-    )
-    (property "Vendor" "C50950" (id 7) (at 265.43 37.465 0)
-      (effects (font (size 1.27 1.27)) hide)
-    )
-    (pin "1")
-    (pin "2")
-    (pin "3")
-    (pin "4")
-    (pin "5")
-  )
   (symbol (lib_id "power:+5V") (at 98.044 35.56 0) (unit 1)
