File: Esquematicos/CAE32_PCB/Pedals/Pedals/Connectors.kicad_sch (KiCad schematic)
At the start: 7 parts, among them J15 USB_C_Receptacle_USB2.0, J16 UART_PGR

Commit message: chore: arrange schematics components
Parts:
- F1: footprint Fuse:Fuse_0603_1608Metric_Pad1.05x0.95mm_HandSolder -> Fuse:Fuse_0603_1608Metric
- R5, R6: footprint Resistor_SMD:R_0603_1608Metric_Pad0.98x0.95mm_HandSolder -> Resistor_SMD:R_0603_1608Metric
Other:
- note added: "USB-C HID PORT"

Commit message: update: PCB pedals Version:2.1.1
Parts:
- removed J16: UART_PGR, Connector_PinSocket_2.54mm:PinSocket_1x05_P2.54mm_Vertical, symbol Connector:Conn_01x05_Female
Connections:
- no-connect marks 3 -> 2
Other:
- note removed: "Programming an Debugging port"
Changed lines of the file:
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@@
   )
   (no_connect (at 56.515 66.04))
-  (no_connect (at 242.57 31.115))
   (no_connect (at 56.515 63.5))
   (wire (pts (xy 78.994 55.88) (xy 87.376 55.88))
@@
     (stroke (width 0) (type default))
   )
-  (polyline (pts (xy 261.62 15.24) (xy 261.62 54.61))
-    (stroke (width 0) (type default))
-  )
   (wire (pts (xy 81.534 35.56) (xy 87.122 35.56))
     (stroke (width 0) (type default))
@@
     (stroke (width 0) (type default))
   )
-  (wire (pts (xy 242.57 33.655) (xy 243.84 33.655))
-    (stroke (width 0) (type default))
-  )
   (wire (pts (xy 56.515 53.34) (xy 87.376 53.34))
     (stroke (width 0) (type default))
@@
     (stroke (width 0) (type default))
   )
-  (wire (pts (xy 243.84 41.275) (xy 242.57 41.275))
-    (stroke (width 0) (type default))
-  )
   (wire (pts (xy 33.655 73.66) (xy 33.655 74.93))
     (stroke (width 0) (type default))
   )
-  (polyline (pts (xy 224.79 54.864) (xy 261.62 54.61))
-    (stroke (width 0) (type default))
-  )
   (polyline (pts (xy 109.22 21.59) (xy 109.22 92.71))
     (stroke (width 0) (type default))
   )
-  (polyline (pts (xy 224.79 15.24) (xy 224.79 54.864))
-    (stroke (width 0) (type default))
-  )
-  (polyline (pts (xy 224.79 15.24) (xy 261.62 15.24))
-    (stroke (width 0) (type default))
-  )
   (wire (pts (xy 70.485 43.18) (xy 74.93 43.18))
     (stroke (width 0) (type default))
@@
     (stroke (width 0) (type default))
   )
-  (wire (pts (xy 243.84 43.815) (xy 243.84 41.275))
-    (stroke (width 0) (type default))
-  )
   (wire (pts (xy 94.742 35.56) (xy 98.044 35.56))
     (stroke (width 0) (type default))
@@
   )
   (wire (pts (xy 56.515 50.8) (xy 73.914 50.8))
-    (stroke (width 0) (type default))
-  )
-  (wire (pts (xy 243.84 33.655) (xy 243.84 29.845))
     (stroke (width 0) (type default))
   )
@@
     (effects (font (size 1.27 1.27)) (justify left bottom))
   )
-  (text "Programming an\nDebugging port" (at 243.205 20.955 0)
-    (effects (font (size 1.27 1.27)) (justify left bottom))
-  )
-  (hierarchical_label "PGR_UART_TX" (shape output) (at 242.57 36.195 0) (fields_autoplaced)
-    (effects (font (size 1.27 1.27)) (justify left))
-  )
   (hierarchical_label "D-" (shape input) (at 87.376 48.26 0) (fields_autoplaced)
-    (effects (font (size 1.27 1.27)) (justify left))
-  )
-  (hierarchical_label "PGR_UART_RX" (shape input) (at 242.57 38.735 0) (fields_autoplaced)
     (effects (font (size 1.27 1.27)) (justify left))
   )
@@
         (path "/f7125cb5-36d2-45a1-8b27-e8e6da0abb82/db5b5259-db1d-46d2-b339-880df6aa32fe"
           (reference "#PWR043") (unit 1)
-        )
-      )
-    )
-  )
-  (symbol (lib_id "power:GNDREF") (at 243.84 43.815 0) (unit 1)
-    (in_bom yes) (on_board yes) (dnp no) (fields_autoplaced)
-    (property "Reference" "#PWR046" (at 243.84 50.165 0)
-      (effects (font (size 1.27 1.27)) hide)
-    )
-    (property "Value" "GNDREF" (at 243.84 48.895 0)
-      (effects (font (size 1.27 1.27)))
-    )
-    (property "Footprint" "" (at 243.84 43.815 0)
-      (effects (font (size 1.27 1.27)) hide)
-    )
-    (property "Datasheet" "" (at 243.84 43.815 0)
-      (effects (font (size 1.27 1.27)) hide)
-    )
-    (pin "1")
-    (instances
-      (project "Pedals"
-        (path "/f7125cb5-36d2-45a1-8b27-e8e6da0abb82/db5b5259-db1d-46d2-b339-880df6aa32fe"
-          (reference "#PWR046") (unit 1)
-        )
-      )
-    )
-  )
-  (symbol (lib_id "power:+3.3V") (at 243.84 29.845 0) (unit 1)
-    (in_bom yes) (on_board yes) (dnp no) (fields_autoplaced)
-    (property "Reference" "#PWR045" (at 243.84 33.655 0)
-      (effects (font (size 1.27 1.27)) hide)
-    )
-    (property "Value" "+3.3V" (at 243.84 24.765 0)
-      (effects (font (size 1.27 1.27)))
-    )
-    (property "Footprint" "" (at 243.84 29.845 0)
-      (effects (font (size 1.27 1.27)) hide)
-    )
-    (property "Datasheet" "" (at 243.84 29.845 0)
-      (effects (font (size 1.27 1.27)) hide)
-    )
-    (pin "1")
-    (instances
-      (project "Pedals"
-        (path "/f7125cb5-36d2-45a1-8b27-e8e6da0abb82/db5b5259-db1d-46d2-b339-880df6aa32fe"
-          (reference "#PWR045") (unit 1)
         )
       )
@@
         )
       )
-    )
-  )
-  (symbol (lib_id "Connector:Conn_01x05_Female") (at 237.49 36.195 180) (unit 1)
-    (in_bom yes) (on_board yes) (dnp no)
-    (property "Reference" "J16" (at 236.22 37.4651 0)
-      (effects (font (size 1.27 1.27)) (justify left))
-    )
-    (property "Value" "UART_PGR" (at 236.22 34.9251 0)
-      (effects (font (size 1.27 1.27)) (justify left))
-    )
-    (property "Footprint" "Connector_PinSocket_2.54mm:PinSocket_1x05_P2.54mm_Vertical" (at 237.49 36.195 0)
-      (effects (font (size 1.27 1.27)) hide)
-    )
-    (property "Datasheet" "~" (at 237.49 36.195 0)
-      (effects (font (size 1.27 1.27)) hide)
-    )
-    (property "LCSC_PART" "C50950" (at 237.49 36.195 0)
-      (effects (font (size 1.27 1.27)) hide)
-    )
-    (property "Item" "C50950" (at 237.49 36.195 0)
-      (effects (font (size 1.27 1.27)) hide)
-    )
-    (property "Qty" "1" (at 237.49 36.195 0)
-      (effects (font (size 1.27 1.27)) hide)
-    )
-    (property "Vendor" "C50950" (at 237.49 36.195 0)
-      (effects (font (size 1.27 1.27)) hide)
-    )
-    (pin "1")
-    (pin "2")
-    (pin "3")
-    (pin "4")
-    (pin "5")
-    (instances
-      (project "Pedals"
-        (path "/f7125cb5-36d2-45a1-8b27-e8e6da0abb82/db5b5259-db1d-46d2-b339-880df6aa32fe"
-          (reference "J16") (unit 1)
-        )
-      )
