File: Esquematicos/CAE32_PCB/Pedals/Pedals/Pedals.kicad_sch (KiCad schematic)
At the start: 32 parts, among them U1 STM32G070RBT6, U2 LDL1117, U4 STM32F072RBTx

Commit message: chore: se corrigen valores de referencias de componentes, creación de nuevas hojas de diagramas, mejor distribución de componentes
Parts:
- removed ST-LINK1, UART_PGRM1: Conn_01x05_Female, Connector_PinHeader_2.54mm:PinHeader_1x05_P2.54mm_Vertical, symbol Connector:Conn_01x05_Female
- removed U1: STM32G070RBT6, Package_QFP:LQFP-32_7x7mm_P0.8mm, symbol MCU_ST_STM32G0:STM32G071KxT
- D: renamed from ID2; value LED -> LED_2
- D: renamed from ID3; value LED -> LED_3
- D: renamed from ID1; value LED -> LED_1
- D: renamed from PWD1; value LED -> PWR
- J5: renamed from DATA1; value 8P8C_LED_Shielded -> PGRM and SPI
- SW1: renamed from BOOT1; value SW_Push -> BOOT
- SW2: renamed from RST1; value SW_Push -> RST
- SW3: renamed from MODE1; value SW_Push -> MODE
- renumbered BRAKE1 to J1, BRAKE2 to J2, ACCEL1 to J3, ACCEL2 to J4, CLUTCH1 to J6, CLUTCH2 to J7, GND1 to TP1, 5V1 to TP2, 3v3 to TP3, U4 to U1
Connections:
- net PSK: no longer U1.50 (PA15)
- net sd: no longer U1.57 (PB5)
- no-connect marks 1 -> 0
Other:
- added sheet Connectors(USB,Programming and debugging) (Connectors.kicad_sch)
- sheet ADCs components ports: added none; removed PSK, agnd, l_s, n_d
- note added: "Pedals SMD's solder point"
- note added: "Power sources test points"
- note removed: "Change actual buttons for the next piece number C2834890"
- note removed: "Power source 5v"
- note removed: "ST-Link Connection"
- note removed: "UART PGRM"
- moved on the sheet: C1, C2, C3, D, J2, J4, J7, R1, R2, R3, R4, SW1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

Commit message: update: Primera revision de etapa ADC lista, ademas de una mejor distrubucion de componentes
Parts:
- removed C1: 100nf, Capacitor_SMD:C_0805_2012Metric_Pad1.18x1.45mm_HandSolder, symbol Device:C_Small
- removed C2, C5: 4.7uf, Capacitor_SMD:C_0805_2012Metric_Pad1.18x1.45mm_HandSolder, symbol Device:C_Small
- removed C4: 1uf, Capacitor_SMD:C_0805_2012Metric_Pad1.18x1.45mm_HandSolder, symbol Device:C_Small
- removed D: PWR, LED_SMD:LED_0805_2012Metric_Pad1.15x1.40mm_HandSolder, symbol Device:LED
- removed J1, J3, J6: Conn_01x03_Female, Connector_PinSocket_2.54mm:PinSocket_1x03_P2.54mm_Vertical, symbol Connector:Conn_01x03_Female
- removed J2, J4, J7: Conn_01x03_Female, Extra_components:1x3_pin, symbol Connector:Conn_01x03_Female
- removed R5: 43, Resistor_SMD:R_0805_2012Metric_Pad1.20x1.40mm_HandSolder, symbol Device:R_Small_US
- removed TP1: GND, TestPoint:TestPoint_Pad_D3.0mm, symbol Connector:TestPoint
- removed TP2: 5v, TestPoint:TestPoint_Pad_D3.0mm, symbol Connector:TestPoint
- removed TP3: 3v3, TestPoint:TestPoint_Pad_D3.0mm, symbol Connector:TestPoint
- removed U2: LDL1117, Package_TO_SOT_SMD:SOT-223-3_TabPin2, symbol Regulator_Linear:AP1117-33
- renumbered C3 to C1, D to D1, D to D2, D to D3, J5 to J1, R2 to R1, R3 to R2, R4 to R3, R1 to R4, SW3 to SW2, SW2 to SW3
Connections:
- net +3.3V: now also SW1.2; no longer SW1.1
- net BOOT: now also R4.1, SW1.1, U1.60 (BOOT0)
- net NRST: now also U1.7 (NRST)
- net SWCLK: no longer R4.1, SW1.2
Other:
- added sheet Power Supply (Power.kicad_sch)
- sheet ADCs components ports: added CS, DIN, DOUT, SCLK; removed none
- sheet Connectors(USB,Programming and debugging) ports: added D+, D-; removed none
- note removed: "Pedals SMD's solder point"
- note removed: "Pedals's Pin Socket"
- note removed: "Power Indicator"
- note removed: "Power sources test points"
- note removed: "STM's power supply"
- company: Techtep -> (none)
- moved on the sheet: C1, R4, SW1, SW2, SW3, U1

Commit message: update: se añade otra hoja para las celdas de carga, ademas de reorganizar todas las hojas
Parts:
- added J1: SPI_MASTER, Connector_PinSocket_2.54mm:PinSocket_1x05_P2.54mm_Horizontal, symbol Connector:Conn_01x05_Female
- added SW2: B2, Button_Switch_SMD:SW_Push_1P1T_NO_6x6mm_H9.5mm, symbol Switch:SW_Push
- added SW3: B3, Button_Switch_SMD:SW_Push_1P1T_NO_6x6mm_H9.5mm, symbol Switch:SW_Push
- C1: footprint Capacitor_SMD:C_0805_2012Metric_Pad1.18x1.45mm_HandSolder -> Capacitor_SMD:C_0603_1608Metric_Pad1.08x0.95mm_HandSolder
- SW1: renamed from SW2; value MODE -> B1
- renumbered J1 to J2, SW1 to SW4, SW3 to SW5
Connections:
- net CS_PDL is gone; now on net S_CS_PEDALS: J2.6
- net IND0 is gone; now on net IND3: R1.1
- net MISO is gone; now on net S_DOUT: J2.4
- net MODE is gone; now on net B1: SW1.1
- net GNDREF: now also J1.1 (Pin_1), SW2.2, SW3.2
- net IND1: now also U1.8 (PC0)
- net IND2: now also U1.9 (PC1)
- net Power Supply/VDD: now also U1.19 (VDD), U1.32 (VDD), U1.64 (VDD)
- net Power Supply/VDDA: now also U1.13 (VDDA)
- net Power Supply/VDDIO2: now also U1.48 (VDDIO2)
- net SCKL: now also U1.21 (PA5), J1.4 (Pin_4); no longer J2.8
- net UART_RX: now also U1.24 (PC4)
- net UART_TX: now also U1.25 (PC5)
- net S_DIN: now reaches J2.5
- net S_DIN: now also U1.11 (PC3)
- net IND3: now reaches U1.10 (PC2)
- net LOAD_CELL_CLK: now reaches U1.14 (PA0)
- net CS_ADC: now reaches U1.20 (PA4)
- net CS_ADC: now also J1.5 (Pin_5)
- net DOUT: now reaches U1.22 (PA6)
- net DOUT: now also J1.3 (Pin_3)
- net DIN: now reaches U1.23 (PA7)
- net DIN: now also J1.2 (Pin_2)
- net LOAD_CELL_3: now reaches U1.26 (PB0)
- net S_CKL: now reaches U1.29 (PB10)
- net S_CKL: now also J2.8
- net S_CS_PEDALS: now reaches U1.33 (PB12)
- net S_DOUT: now reaches U1.35 (PB14)
- net LOAD_CELL_2: now reaches U1.37 (PC6)
- net LOAD_CELL_1: now reaches U1.38 (PC7)
- net B3: now reaches U1.39 (PC8)
- net B3: now also SW3.1
- net B2: now reaches U1.40 (PC9)
- net B2: now also SW2.1
- net B1: now reaches U1.41 (PA8)
- net PGR_UART_RX: now reaches U1.42 (PA9)
- net PGR_UART_TX: now reaches U1.43 (PA10)
- net D-: now reaches U1.44 (PA11)
- net D+: now reaches U1.45 (PA12)
- net CAN_RX: now reaches U1.61 (PB8)
- net CAN_TX: now reaches U1.62 (PB9)
- net MOSI: no longer names the net of J2.2
Other:
- added sheet Load Cells (Load_cells.kicad_sch)
- sheet Connectors(USB,Programming and debugging) ports: added PGR_UART_RX, PGR_UART_TX; removed USART_RX, USART_TX
- note added: "MISC buttons"
- note added: "Reset and boot buttons"
- note added: "SPI_MASTER"
- note removed: "Activate Update Mode"
- moved on the sheet: C1, R4, SW1, SW4, SW5

Commit message: update: Componentes acomodados en la PCB
Parts:
- removed SW1: B1, Button_Switch_SMD:SW_Push_1P1T_NO_6x6mm_H9.5mm, symbol Switch:SW_Push
- removed SW2: B2, Button_Switch_SMD:SW_Push_1P1T_NO_6x6mm_H9.5mm, symbol Switch:SW_Push
- removed SW3: B3, Button_Switch_SMD:SW_Push_1P1T_NO_6x6mm_H9.5mm, symbol Switch:SW_Push
- added H1, H2, H3, H4: M, MountingHole:MountingHole_3.2mm_M3_Pad_Via, symbol Mechanical:MountingHole_Pad
- added J2: Conn_01x02_Male, Connector_PinHeader_2.54mm:PinHeader_1x02_P2.54mm_Vertical, symbol Connector:Conn_01x02_Male
- added SW1: CONFIG, Button_Switch_SMD:SW_DIP_SPSTx03_Slide_6.7x9.18mm_W6.73mm_P2.54mm_LowProfile_JPin, symbol Switch:SW_DIP_x03
- R1, R2, R3, R4: footprint Resistor_SMD:R_0805_2012Metric_Pad1.20x1.40mm_HandSolder -> Resistor_SMD:R_0603_1608Metric_Pad0.98x0.95mm_HandSolder
- renumbered J2 to J3, SW4 to SW2, SW5 to SW3
Connections:
- net B1: now also SW1.4
- net B2: now also SW1.5
- net B3: now also SW1.6
- net CAN_RX: now also J2.1 (Pin_1)
- net CAN_TX: now also J2.2 (Pin_2)
- net GNDREF: now also U1.12 (VSSA), U1.18 (VSS), U1.31 (VSS), U1.47 (VSS), U1.63 (VSS), H1.1, H2.1, H3.1, H4.1, SW1.1, SW1.2, SW1.3
Other:
- note added: "DIP config switches"
- note added: "Mounting Holes"
- note added: "SPI Master and CAN PORT"
- note removed: "MISC buttons"
- moved on the sheet: J1

Commit message: update: se agrega el consumo de corriente a los IC's ademas de agregar el URL y numero de parte de los componentes de LCSC en kicad
Parts:
- C1: value 0.1uf -> 100n; LCSC_PART (none) -> c1591
- D1: value LED_1 -> LED; LCSC_PART (none) -> C965815
- D2: value LED_2 -> LED; LCSC_PART (none) -> C965815
- D3: value LED_3 -> LED; LCSC_PART (none) -> C965815
- J1: LCSC_PART (none) -> C50950
- J2: value Conn_01x02_Male -> CAN; LCSC_PART (none) -> C492401
- J3: LCSC_PART (none) -> C386757
- R1, R2, R3: value 10 -> 330; LCSC_PART (none) -> C25804
- R4: LCSC_PART (none) -> C25804
- SW1: footprint Button_Switch_SMD:SW_DIP_SPSTx03_Slide_6.7x9.18mm_W6.73mm_P2.54mm_LowProfile_JPin -> Button_Switch_SMD:SW_DIP_SPSTx03_Slide_KingTek_DSHP03TJ_W5.25mm_P1.27mm_JPin; LCSC_PART (none) -> C5289932
- SW2, SW3: LCSC_PART (none) -> C2834890
- U1: LCSC_PART (none) -> C46046
Other:
- note added: "Total current into sum of all VDD power lines 120mA External main supply voltage: MIN:-0.3v MAX:4.0v"
- moved on the sheet: U1

Commit message: Update: esquematicos de PCB, reorganizando elementos para hacer mas compacta la pcb, ademas de agregar serigrafia e imagenes de la PCB
Parts:
- H1, H2, H3, H4: footprint MountingHole:MountingHole_3.2mm_M3_Pad_Via -> MountingHole:MountingHole_2.2mm_M2_DIN965_Pad
- J1: footprint Connector_PinSocket_2.54mm:PinSocket_1x05_P2.54mm_Horizontal -> Connector_PinSocket_2.54mm:PinSocket_1x05_P2.54mm_Vertical
Changed lines of the file:
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@@
       (effects (font (size 1.27 1.27)) (justify left))
     )
-    (property "Footprint" "MountingHole:MountingHole_3.2mm_M3_Pad_Via" (id 2) (at 266.065 149.86 0)
+    (property "Footprint" "MountingHole:MountingHole_2.2mm_M2_DIN965_Pad" (id 2) (at 266.065 149.86 0)
       (effects (font (size 1.27 1.27)) hide)
     )
@@
       (effects (font (size 1.27 1.27)) (justify left))
     )
-    (property "Footprint" "MountingHole:MountingHole_3.2mm_M3_Pad_Via" (id 2) (at 250.19 149.86 0)
+    (property "Footprint" "MountingHole:MountingHole_2.2mm_M2_DIN965_Pad" (id 2) (at 250.19 149.86 0)
       (effects (font (size 1.27 1.27)) hide)
     )
@@
       (effects (font (size 1.27 1.27)) (justify left))
     )
-    (property "Footprint" "MountingHole:MountingHole_3.2mm_M3_Pad_Via" (id 2) (at 255.905 149.86 0)
+    (property "Footprint" "MountingHole:MountingHole_2.2mm_M2_DIN965_Pad" (id 2) (at 255.905 149.86 0)
       (effects (font (size 1.27 1.27)) hide)
     )
@@
       (effects (font (size 1.27 1.27)) (justify left))
     )
-    (property "Footprint" "MountingHole:MountingHole_3.2mm_M3_Pad_Via" (id 2) (at 260.985 149.86 0)
+    (property "Footprint" "MountingHole:MountingHole_2.2mm_M2_DIN965_Pad" (id 2) (at 260.985 149.86 0)
       (effects (font (size 1.27 1.27)) hide)
     )
@@
     (property "Reference" "J1" (id 0) (at 192.405 119.38 0))
     (property "Value" "SPI_MASTER" (id 1) (at 192.405 121.92 0))
-    (property "Footprint" "Connector_PinSocket_2.54mm:PinSocket_1x05_P2.54mm_Horizontal" (id 2) (at 191.77 130.175 0)
+    (property "Footprint" "Connector_PinSocket_2.54mm:PinSocket_1x05_P2.54mm_Vertical" (id 2) (at 191.77 130.175 0)
       (effects (font (size 1.27 1.27)) hide)
     )
@@
     )
     (path "/24d197b5-8acb-4d99-8e5d-25048dd62849"
-      (reference "H1") (unit 1) (value "M") (footprint "MountingHole:MountingHole_3.2mm_M3_Pad_Via")
+      (reference "H1") (unit 1) (value "M") (footprint "MountingHole:MountingHole_2.2mm_M2_DIN965_Pad")
     )
     (path "/3973bfc9-bcd6-4f06-8ccc-37dab1d0c469"
-      (reference "H2") (unit 1) (value "M") (footprint "MountingHole:MountingHole_3.2mm_M3_Pad_Via")
+      (reference "H2") (unit 1) (value "M") (footprint "MountingHole:MountingHole_2.2mm_M2_DIN965_Pad")
     )
     (path "/930eb733-a967-4793-9d84-fdf5e0d67f86"
-      (reference "H3") (unit 1) (value "M") (footprint "MountingHole:MountingHole_3.2mm_M3_Pad_Via")
+      (reference "H3") (unit 1) (value "M") (footprint "MountingHole:MountingHole_2.2mm_M2_DIN965_Pad")
     )
     (path "/2464bc3f-5269-4b31-a1c1-48b0deb8f337"
-      (reference "H4") (unit 1) (value "M") (footprint "MountingHole:MountingHole_3.2mm_M3_Pad_Via")
+      (reference "H4") (unit 1) (value "M") (footprint "MountingHole:MountingHole_2.2mm_M2_DIN965_Pad")
     )
     (path "/db448617-4c4d-4414-b908-dcf012a48abf"
-      (reference "J1") (unit 1) (value "SPI_MASTER") (footprint "Connector_PinSocket_2.54mm:PinSocket_1x05_P2.54mm_Horizontal")
+      (reference "J1") (unit 1) (value "SPI_MASTER") (footprint "Connector_PinSocket_2.54mm:PinSocket_1x05_P2.54mm_Vertical")
     )
     (path "/6a9f9c80-ce4e-45f4-a95d-764bf4249ff8"
@@
     )
     (path "/db5b5259-db1d-46d2-b339-880df6aa32fe/d9aacc9d-05ae-4825-9a0d-6ffb9e4a0908"
-      (reference "J16") (unit 1) (value "UART_PGR") (footprint "Connector_PinSocket_2.54mm:PinSocket_1x05_P2.54mm_Horizontal")
+      (reference "J16") (unit 1) (value "UART_PGR") (footprint "Connector_PinSocket_2.54mm:PinSocket_1x05_P2.54mm_Vertical")
     )
     (path "/db5b5259-db1d-46d2-b339-880df6aa32fe/edba0ae9-c38d-42f3-b7ef-6a137906c1bd"
-      (reference "J17") (unit 1) (value "ST-Link") (footprint "Connector_PinSocket_2.54mm:PinSocket_1x05_P2.54mm_Horizontal")
+      (reference "J17") (unit 1) (value "ST-Link") (footprint "Connector_PinSocket_2.54mm:PinSocket_1x05_P2.54mm_Vertical")
     )
     (path "/d0544081-4d46-4bd0-961b-9683f35d3586/5645bbe1-320e-4607-a8c9-ca2df583753a"
@@
     )
     (path "/af4de2bd-7a38-4d95-b043-2fd3b0e6e25e/3c755e88-f94d-4eee-9da7-b5b9c94f38e4"
-      (reference "TP1") (unit 1) (value "GND") (footprint "TestPoint:TestPoint_Pad_D3.0mm")
+      (reference "TP1") (unit 1) (value "GND") (footprint "TestPoint:TestPoint_Pad_D1.0mm")
     )
     (path "/af4de2bd-7a38-4d95-b043-2fd3b0e6e25e/36533663-7998-4304-8c67-fce0d7b1fd0c"
-      (reference "TP2") (unit 1) (value "5v") (footprint "TestPoint:TestPoint_Pad_D3.0mm")
+      (reference "TP2") (unit 1) (value "5v") (footprint "TestPoint:TestPoint_Pad_D1.0mm")
     )
     (path "/af4de2bd-7a38-4d95-b043-2fd3b0e6e25e/2f7d23da-5592-4647-a7f1-21a65883ff4a"
-      (reference "TP3") (unit 1) (value "3v3") (footprint "TestPoint:TestPoint_Pad_D3.0mm")
+      (reference "TP3") (unit 1) (value "3v3") (footprint "TestPoint:TestPoint_Pad_D1.0mm")
+    )
+    (path "/d0544081-4d46-4bd0-961b-9683f35d3586/e9c93b4d-9b20-47f9-ad09-1c5b42809e01"
+      (reference "TP4") (unit 1) (value "TestPoint") (footprint "TestPoint:TestPoint_Pad_D1.0mm")
+    )
+    (path "/d0544081-4d46-4bd0-961b-9683f35d3586/ab5c869d-6fec-4307-b52a-a0a0a3ba65ae"
+      (reference "TP5") (unit 1) (value "TestPoint") (footprint "TestPoint:TestPoint_Pad_D1.0mm")
+    )
+    (path "/d0544081-4d46-4bd0-961b-9683f35d3586/c032cbe9-fa28-4b72-a603-fb3cc494b270"
+      (reference "TP6") (unit 1) (value "TestPoint") (footprint "TestPoint:TestPoint_Pad_D1.0mm")
+    )
+    (path "/d0544081-4d46-4bd0-961b-9683f35d3586/55466aec-0a20-4387-9a6b-9e4c0cb6c611"
+      (reference "TP7") (unit 1) (value "TestPoint") (footprint "TestPoint:TestPoint_Pad_D1.0mm")
     )
     (path "/beb69fcb-f032-45d6-a522-3b1db9902ca2"

Commit message: update: se crea la primera revisión de la PCB
Parts:
- C1: Item (none) -> c1591; Qty (none) -> 22; Vendor (none) -> c1591
- D1, D2, D3: Item (none) -> C965815; Qty (none) -> 4; Vendor (none) -> C965815
- H1, H2, H3, H4: Qty (none) -> 4
- J1: Item (none) -> C50950; Qty (none) -> 1; Vendor (none) -> C50950
- J2: Item (none) -> C492401; Qty (none) -> 1; Vendor (none) -> C492401
- J3: Item (none) -> C386757; Qty (none) -> 1; Vendor (none) -> C386757
- R1, R2, R3: Item (none) -> C25804; Qty (none) -> 4; Vendor (none) -> C25804
- R4: Item (none) -> C25804; Qty (none) -> 1; Vendor (none) -> C25804
- SW1: Item (none) -> C5289932; Qty (none) -> 1; Vendor (none) -> C5289932
- SW2, SW3: Item (none) -> C2834890; Qty (none) -> 1; Vendor (none) -> C2834890
- U1: Item (none) -> C46046; Qty (none) -> 1; Vendor (none) -> C46046

Commit message: add: plantilla para diseño de pcb para shifter
Changed lines of the file:
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@@
     (effects (font (size 1.27 1.27)) (justify left bottom))
-  )
-  (label "SWDIO" (at 125.73 172.72 180)
-    (effects (font (size 1.27 1.27)) (justify right bottom))
   )
   (label "S_CS_PEDALS" (at 265.43 38.1 0)
@@
   )
   (label "NRST" (at 30.48 47.625 180)
-    (effects (font (size 1.27 1.27)) (justify right bottom))
-  )
-  (label "SWCLK" (at 125.73 168.91 180)
     (effects (font (size 1.27 1.27)) (justify right bottom))
   )
@@
       (reference "#PWR046") (unit 1) (value "GNDREF") (footprint "")
     )
-    (path "/db5b5259-db1d-46d2-b339-880df6aa32fe/94064232-2224-4afe-b3f9-65089df96c73"
-      (reference "#PWR047") (unit 1) (value "+3.3V") (footprint "")
-    )
-    (path "/db5b5259-db1d-46d2-b339-880df6aa32fe/37ddbbab-607b-45c8-9507-05ab3854d485"
-      (reference "#PWR048") (unit 1) (value "GNDREF") (footprint "")
-    )
     (path "/af4de2bd-7a38-4d95-b043-2fd3b0e6e25e/22032096-7e65-4bdc-a0d3-7b58c55da033"
       (reference "#PWR049") (unit 1) (value "GNDREF") (footprint "")
@@
       (reference "J16") (unit 1) (value "UART_PGR") (footprint "Connector_PinSocket_2.54mm:PinSocket_1x05_P2.54mm_Vertical")
     )
-    (path "/db5b5259-db1d-46d2-b339-880df6aa32fe/edba0ae9-c38d-42f3-b7ef-6a137906c1bd"
-      (reference "J17") (unit 1) (value "ST-Link") (footprint "Connector_PinSocket_2.54mm:PinSocket_1x05_P2.54mm_Vertical")
-    )
     (path "/d0544081-4d46-4bd0-961b-9683f35d3586/5645bbe1-320e-4607-a8c9-ca2df583753a"
