File: Esquematicos/CAE32_PCB/Pedals/Pedals/ADC.kicad_sch (KiCad schematic)
At the start: 16 parts, among them J10 Conn_01x03_Female, J11 Conn_01x03_Female, J12 Conn_01x03_Female, J13 Conn_01x03_Female, J14 Conn_01x03_Female, J4 Conn_01x03_Female, J5 Conn_01x03_Female, J6 Conn_01x03_Female, J7 Conn_01x03_Female, J8 Conn_01x03_Female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

Commit message: update: PCB pedals Version:2.1.1
Parts:
- removed J12, J4, J8: Conn_01x03_Female, Connector_PinSocket_2.54mm:PinSocket_1x03_P2.54mm_Vertical, symbol Connector:Conn_01x03_Female
- added C36, C37, C38, C39, C40, C41, C42, C43: 33n, Capacitor_SMD:C_0603_1608Metric, symbol Device:C
- added R23, R24, R25, R26, R27, R28, R29, R30: 100, Resistor_SMD:R_0603_1608Metric, symbol Device:R_Small_US
- J10, J11, J13, J14, J5, J6, J7, J9: footprint Extra_components:1x3_pin -> Connector_PinHeader_2.54mm:PinHeader_1x03_P2.54mm_Vertical; Item (none) -> C6332196; LCSC_PART (none) -> C6332196; Vendor (none) -> C6332196
Connections:
- net ACCEL: now also R29.1; no longer U3.5 (IN1)
- net BRAKE: now also R30.1; no longer U3.4 (IN0)
- net CLUTCH: now also R26.1; no longer U3.6 (IN2)
- net GNDREF: now also C36.2, C37.2, C38.2, C39.2, C40.2, C41.2, C42.2, C43.2
- net Custom_1 renamed CH_1
- net CH_1: now also R23.1; no longer U3.11 (IN7)
- net Custom_2 renamed CH_2
- net CH_2: now also R24.1; no longer U3.10 (IN6)
- net Custom_3 renamed CH_3
- net CH_3: now also R25.1; no longer U3.9 (IN5)
- net Custom_4 renamed CH_4
- net CH_4: now also R28.1; no longer U3.8 (IN4)
- net Custom_5 renamed CH_5
- net CH_5: now also R27.1; no longer U3.7 (IN3)
- new net IN0: C43.1, R30.2, U3.4 (IN0)
- new net IN1: C42.1, R29.2, U3.5 (IN1)
- new net IN2: C41.1, R28.2, U3.6 (IN2)
- new net IN3: C36.1, R27.2, U3.7 (IN3)
- new net IN4: C37.1, R26.2, U3.8 (IN4)
- new net IN5: C38.1, R25.2, U3.9 (IN5)
- new net IN6: C39.1, R24.2, U3.10 (IN6)
- new net IN7: C40.1, R23.2, U3.11 (IN7)
Other:
- note removed: "Pedals SMD's solder point"
