File: Esquematicos/CAE32_PCB/Pedals/Pedals.kicad_pcb (KiCad board)
At the start: 4 copper layers, 86 x 62 mm, 124 parts, among them J1 Conn_01x19_Pin, J10 Conn_01x03_Female, J11 Conn_01x03_Female, J13 Conn_01x03_Female, J14 Conn_01x03_Female, J15 USB_C_Receptacle_USB2.0, J17 LC, J18 LC, J19 LC, J5 Conn_01x03_Female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

Commit message: chore: Moved all the Pedals contents a folder above and updated pcb including the required oscilator
Parts:
- added C44: 12p, Capacitor_SMD:C_0603_1608Metric, F.Cu at (136.9, 77.5)
- added C45: 12p, Capacitor_SMD:C_0603_1608Metric, F.Cu at (144.8, 75.0)
- added Y1: Crystal_GND24_Small, Crystal:Crystal_SMD_3225-4Pin_3.2x2.5mm, F.Cu at (140.8, 76.5)
Connections:
- U1 pad 24: /UART_RX -> /UART_TX
- U1 pad 25: /UART_TX -> /UART_RX
- U1 pad 42: /PGR_UART_RX -> /PGR_UART_TX
- U1 pad 43: /PGR_UART_TX -> /PGR_UART_RX
- U1 pad 5: unconnected-(U1-PF0-Pad5) -> /OSC_IN
- U1 pad 6: unconnected-(U1-PF1-Pad6) -> /OSC_OUT
Routing:
- net /OSC_OUT: track 0.00 -> 15.3 mm
- net /OSC_IN: track 0.00 -> 15.0 mm
- net GNDREF: track 44.7 -> 54.9 mm, vias 43 -> 48
- net /PGR_UART_RX: track 71.9 -> 69.1 mm
- net /PGR_UART_TX: track 69.3 -> 66.8 mm
- net /BOOT: track 76.0 -> 76.6 mm
Other:
- board text added: "EXPANSION PORT"
