File: Esquematicos/CAE32_PCB/Pedals/Pedals.kicad_sch (KiCad schematic)
At the start: 17 parts, among them J1 Conn_01x19_Pin, SW1 CONFIG, SW2 SW, SW3 SW, U1 STM32F072RBTx

Commit message: chore: Moved all the Pedals contents a folder above and updated pcb including the required oscilator
Parts:
- added C44, C45: 12p, Capacitor_SMD:C_0603_1608Metric, symbol Device:C_Small
- added Y1: Crystal_GND24_Small, Crystal:Crystal_SMD_3225-4Pin_3.2x2.5mm, symbol Device:Crystal_GND24_Small
Connections:
- net GNDREF: now also C44.2, C45.2, Y1.2, Y1.4
- net PGR_UART_RX: now also U1.43 (PA10); no longer U1.42 (PA9)
- net PGR_UART_TX: now also U1.42 (PA9); no longer U1.43 (PA10)
- net UART_RX: now also U1.25 (PC5); no longer U1.24 (PC4)
- net UART_TX: now also U1.24 (PC4); no longer U1.25 (PC5)
- net OSC_IN: now reaches U1.5 (PF0)
- net OSC_IN: now also C45.1, Y1.1
- net OSC_OUT: now reaches U1.6 (PF1)
- net OSC_OUT: now also C44.1, Y1.3
