File: Schematics/CAE32_PCB/Pedals/Load_cells.kicad_sch (KiCad schematic)
At the start: 55 parts, among them J17 LC, J18 LC, J19 LC, Q1 MMBT3906, Q2 MMBT3906, Q3 MMBT3906, U5 HX711, U6 HX711, U7 HX711

Commit message: updated: Pcb design, fixed plane grounds and minor improvements, added stlink connector, updated BOM with the current market stock
Parts:
- C15, C16, C17, C18, C19, C22, C23, C24, C27, C28, C29, C30, C31, C33, C35: Item c1591 -> C66501; LCSC_PART c1591 -> C66501; Vendor c1591 -> C66501
- JP1, JP2, JP3, TP4, TP5, TP6, TP7: now not fitted
- R16, R17, R22: value 10k -> 10K

Commit message: fixed: SPI route
Changed lines of the file:
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@@
 (kicad_sch
-	(version 20231120)
+	(version 20250114)
 	(generator "eeschema")
-	(generator_version "8.0")
+	(generator_version "9.0")
 	(paper "A4")
 	(title_block
@@
 		(comment 2 "Version 2.1")
 	)
+	(text "HX711"
+		(exclude_from_sim no)
+		(at 110.49 17.78 0)
+		(effects
+			(font
+				(size 1.27 1.27)
+				(thickness 0.254)
+				(bold yes)
+			)
+			(justify left bottom)
+		)
+	)
+	(text "SparkFun_HX711_Load_Cell_V11\nDesign by: N.Seidle\nLicense:CC BY-SA 4.0"
+		(exclude_from_sim no)
+		(at 249.555 19.05 0)
+		(effects
+			(font
+				(size 1.27 1.27)
+			)
+			(justify left bottom)
+		)
+	)
+	(text "E+\nE-\nA+\nA-\nB-\nB+\nShield"
+		(exclude_from_sim no)
+		(at 23.114 48.768 0)
+		(effects
+			(font
+				(size 1.27 1.27)
+				(thickness 0.254)
+				(bold yes)
+			)
+			(justify left bottom)
+		)
+	)
+	(text "E+\nE-\nA+\nA-\nB-\nB+\nShield"
+		(exclude_from_sim no)
+		(at 21.59 137.16 0)
+		(effects
+			(font
+				(size 1.27 1.27)
+				(thickness 0.254)
+				(bold yes)
+			)
+			(justify left bottom)
+		)
+	)
+	(text "E+\nE-\nA+\nA-\nB-\nB+\nShield"
+		(exclude_from_sim no)
+		(at 160.147 101.727 0)
+		(effects
+			(font
+				(size 1.27 1.27)
+				(thickness 0.254)
+				(bold yes)
+			)
+			(justify left bottom)
+		)
+	)
+	(text "ANALOG SUPPLY CURRENT: 1400uA\nDIGITAL SUPPLY CURRENT: 100uA"
+		(exclude_from_sim no)
+		(at 110.49 22.225 0)
+		(effects
+			(font
+				(size 1.27 1.27)
+			)
+			(justify left bottom)
+		)
+	)
+	(text "Modifications:\nMerge the two input connectors in to one"
+		(exclude_from_sim no)
+		(at 244.475 25.4 0)
+		(effects
+			(font
+				(size 1.27 1.27)
+			)
+			(justify left bottom)
+		)
+	)
 	(junction
 		(at 100.965 32.385)
@@
 		)
 	)
-	(text "HX711"
-		(exclude_from_sim no)
-		(at 110.49 17.78 0)
-		(effects
-			(font
-				(size 1.27 1.27)
-				(thickness 0.254)
-				(bold yes)
-			)
-			(justify left bottom)
-		)
-	)
-	(text "SparkFun_HX711_Load_Cell_V11\nDesign by: N.Seidle\nLicense:CC BY-SA 4.0"
-		(exclude_from_sim no)
-		(at 249.555 19.05 0)
-		(effects
-			(font
-				(size 1.27 1.27)
-			)
-			(justify left bottom)
-		)
-	)
-	(text "E+\nE-\nA+\nA-\nB-\nB+\nShield"
-		(exclude_from_sim no)
-		(at 23.114 48.768 0)
-		(effects
-			(font
-				(size 1.27 1.27)
-				(thickness 0.254)
-				(bold yes)
-			)
-			(justify left bottom)
-		)
-	)
-	(text "E+\nE-\nA+\nA-\nB-\nB+\nShield"
-		(exclude_from_sim no)
-		(at 21.59 137.16 0)
-		(effects
-			(font
-				(size 1.27 1.27)
-				(thickness 0.254)
-				(bold yes)
-			)
-			(justify left bottom)
-		)
-	)
-	(text "E+\nE-\nA+\nA-\nB-\nB+\nShield"
-		(exclude_from_sim no)
-		(at 160.147 101.727 0)
-		(effects
-			(font
-				(size 1.27 1.27)
-				(thickness 0.254)
-				(bold yes)
-			)
-			(justify left bottom)
-		)
-	)
-	(text "ANALOG SUPPLY CURRENT: 1400uA\nDIGITAL SUPPLY CURRENT: 100uA"
-		(exclude_from_sim no)
-		(at 110.49 22.225 0)
-		(effects
-			(font
-				(size 1.27 1.27)
-			)
-			(justify left bottom)
-		)
-	)
-	(text "Modifications:\nMerge the two input connectors in to one"
-		(exclude_from_sim no)
-		(at 244.475 25.4 0)
-		(effects
-			(font
-				(size 1.27 1.27)
-			)
-			(justify left bottom)
-		)
-	)
 	(label "B2+"
 		(at 35.56 135.89 0)
-		(fields_autoplaced yes)
 		(effects
 			(font
@@
 	(label "A1+"
 		(at 37.465 40.005 0)
-		(fields_autoplaced yes)
 		(effects
 			(font
@@
 	(label "B2+"
 		(at 88.9 149.86 180)
-		(fields_autoplaced yes)
 		(effects
 			(font
@@
 	(label "B3-"
 		(at 227.33 116.84 180)
-		(fields_autoplaced yes)
 		(effects
 			(font
@@
 	(label "A2-"
 		(at 45.72 154.94 180)
-		(fields_autoplaced yes)
 		(effects
 			(font
@@
 	(label "B2-"
 		(at 88.9 152.4 180)
-		(fields_autoplaced yes)
 		(effects
 			(font
@@
 	(label "A3-"
 		(at 173.99 95.25 0)
-		(fields_autoplaced yes)
 		(effects
 			(font
@@
 	(label "B1-"
 		(at 37.465 45.085 0)
-		(fields_autoplaced yes)
 		(effects
 			(font
@@
 	(label "B3+"
 		(at 227.33 114.3 180)
-		(fields_autoplaced yes)
 		(effects
 			(font
@@
 	(label "A2+"
 		(at 35.56 128.27 0)
-		(fields_autoplaced yes)
 		(effects
 			(font
@@
 	(label "A1-"
 		(at 37.465 42.545 0)
-		(fields_autoplaced yes)
 		(effects
 			(font
@@
 	(label "B2-"
 		(at 35.56 133.35 0)
-		(fields_autoplaced yes)
 		(effects
 			(font
@@
 	(label "B3+"
 		(at 173.99 100.33 0)
-		(fields_autoplaced yes)
 		(effects
 			(font
@@
 	(label "A1-"
 		(at 47.625 66.675 180)
-		(fields_autoplaced yes)
 		(effects
 			(font
@@
 	(label "B3-"
 		(at 173.99 97.79 0)
-		(fields_autoplaced yes)
 		(effects
 			(font
@@
 	(label "B1-"
 		(at 90.805 64.135 180)
-		(fields_autoplaced yes)
 		(effects
 			(font
@@
 	(label "A2-"
 		(at 35.56 130.81 0)
-		(fields_autoplaced yes)
 		(effects
 			(font
@@
 	(label "B1+"
 		(at 37.465 47.625 0)
-		(fields_autoplaced yes)
 		(effects
 			(font
@@
 	(label "B1+"
 		(at 90.805 61.595 180)
-		(fields_autoplaced yes)
 		(effects
 			(font
@@
 	(label "A3+"
 		(at 184.15 111.76 180)
-		(fields_autoplaced yes)
 		(effects
 			(font
@@
 	(label "A1+"
 		(at 47.625 59.055 180)
-		(fields_autoplaced yes)
 		(effects
 			(font
@@
 	(label "A3-"
 		(at 184.15 119.38 180)
-		(fields_autoplaced yes)
 		(effects
 			(font
@@
 	(label "A2+"
 		(at 45.72 147.32 180)
-		(fields_autoplaced yes)
 		(effects
 			(font
@@
 	(label "A3+"
 		(at 173.99 92.71 0)
-		(fields_autoplaced yes)
 		(effects
 			(font
@@
 		(shape input)
 		(at 114.3 137.16 0)
-		(fields_autoplaced yes)
 		(effects
 			(font
@@
 		(shape input)
 		(at 135.89 48.895 0)
-		(fields_autoplaced yes)
 		(effects
 			(font
@@
 		(shape output)
 		(at 264.16 99.06 0)
-		(fields_autoplaced yes)
 		(effects
 			(font
@@
 		(shape output)
 		(at 123.19 46.355 0)
-		(fields_autoplaced yes)
 		(effects
 			(font
@@
 		(shape input)
 		(at 252.73 101.6 0)
-		(fields_autoplaced yes)
 		(effects
 			(font
@@
 		(shape output)
 		(at 119.38 134.62 0)
-		(fields_autoplaced yes)
-		(effects
-			(font
+		(effects
+			(font
